File: BLDC_PHOBOS_2021 - ImprovedUpperTraces/BLDC_PHOBOS_2021/PowerPCB.kicad_pcb (KiCad board)
At the start: 4 copper layers, 217 x 100 mm, 276 parts, among them J1 POWER+, J10 +3V3 External, J11 Con_POWER_B+, J12 CommonGND_PowerPCB, J13 CommonGND_ControlPCB, J14 Phase_A_RAW, J15 Con_POWER_GND, J16 Phase_B_RAW, J17 Phase_C_RAW, J18 Low_Battery_Voltage_Indicator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, J19 Phase_A_Zero_Filtered_Start, J2 48V_From_PowerPCB, J20 A_MOS_HIGH_ControlPCB, J21 A_MOS_HIGH_PowerPCB, J22 Power_ON_Indicator_Output, J23 Phase_B_Zero_Filtered_Start, J24 A_MOS_LOW_ControlPCB, J25 Phase_A_PowerPCB, J26 Connector_A, J27 Program&Control_Button, J28 Phase_C_Zero_Filtered_Start, J29 A_MOS_LOW_PowerPCB, J3 48V_to_Control_PCB, J30 Phase_A_ControlPCB, J31 Phase_A_Zero_Filtered_Normal, J32 A_Shunt+_PowerPCB, J33 A_Shunt+_ControlPCB, J34 Phase_B_Zero_Filtered_Normal, J35 Phase_C_Zero_Filtered_Normal, J36 B_MOS_HIGH_PowerPCB, J37 B_MOS_HIGH_ControlPCB, J38 Phase_B_PowerPCB, J39 B_MOS_LOW_ControlPCB, J4 +15V External, J40 Connector_B, J41 Hall +3V3, J42 B_MOS_LOW_PowerPCB, J43 Phase_B_ControlPCB, J44 Con_HALL_A, J45 B_Shunt+_PowerPCB, J46 B_Shunt+_ControlPCB, J47 Con_HALL_B, J48 Con_HALL_C, J49 C_MOS_HIGH_PowerPCB, J5 Total_Current_Differential-_P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, J50 C_MOS_HIGH_ControlPCB, J51 Hall GND, J52 Phase_C_PowerPCB, J53 C_MOS_LOW_ControlPCB, J54 Connector_C, J55 C_MOS_LOW_PowerPCB, J56 Phase_C_ControlPCB, J57 Voltage Sense SGN, J58 C_Shunt+_PowerPCB, J59 C_Shunt+_ControlPCB, J6 Total_Current_Differential-_C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, J60 Total_Battery_Current, J61 A_Low_Side_Current_ADC, J62 B_Low_Side_Current_ADC, J63 C_Low_Side_Current_ADC, J64 Throttle 3V3, J65 Throttle Signal, J66 Throttle GND, J67 A_HIGH_MCU, J68 A_LOW_MCU, J69 B_HIGH_MCU, J7 +5V External, J70 B_LOW_MCU, J71 C_HIGH_MCU, J72 C_LOW_MCU, J73 I2C 3V3, J74 VIN, J75 GND, J76 I2C_SCL, J77 PA2, J78 PA7, J79 PA6, J8 Total_Current_Differential+_P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, J80 PA5, J81 PA4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

Commit message: Updated Design
Parts:
- removed J74: VIN, Connector_PinHeader_2.54mm:PinHeader_1x01_P2.54mm_Vertical
- removed J75: GND, Connector_PinHeader_2.54mm:PinHeader_1x01_P2.54mm_Vertical
- removed J77, J94: PA2, Connector_PinHeader_2.54mm:PinHeader_1x01_P2.54mm_Vertical
- removed J78: PA7, Connector_PinHeader_2.54mm:PinHeader_1x01_P2.54mm_Vertical
- removed J79: PA6, Connector_PinHeader_2.54mm:PinHeader_1x01_P2.54mm_Vertical
- removed J80: PA5, Connector_PinHeader_2.54mm:PinHeader_1x01_P2.54mm_Vertical
- removed J81: PA4, Connector_PinHeader_2.54mm:PinHeader_1x01_P2.54mm_Vertical
- removed J83: PA3, Connector_PinHeader_2.54mm:PinHeader_1x01_P2.54mm_Vertical
- removed J84: PA1, Connector_PinHeader_2.54mm:PinHeader_1x01_P2.54mm_Vertical
- removed J85: PA0, Connector_PinHeader_2.54mm:PinHeader_1x01_P2.54mm_Vertical
- removed J87, J95: 3V3, Connector_PinHeader_2.54mm:PinHeader_1x01_P2.54mm_Vertical
- removed J88: PB3, Connector_PinHeader_2.54mm:PinHeader_1x01_P2.54mm_Vertical
- removed J90: Motor_Temp, Connector_PinHeader_2.54mm:PinHeader_1x01_P2.54mm_Vertical
- moved J72 29.8 mm to (276.3, 85.7), turned to 90 degrees
- moved C32 27.3 mm to (296.4, 51.3), turned to 90 degrees
- moved J57 26.2 mm to (300.8, 73.9), turned to 270 degrees
- moved D3 25.8 mm to (291.4, 100.0), turned to 90 degrees
- moved J70 25.6 mm to (276.3, 82.5), turned to 90 degrees
- moved J60 24.2 mm to (298.4, 56.8), turned to 270 degrees
- moved U80 23.7 mm to (287.3, 99.0), turned to 270 degrees
- moved U21 23.7 mm to (278.9, 50.1), turned to 0 degrees
- moved R25 21.9 mm to (297.4, 73.9), turned to 0 degrees
- moved J68 21.7 mm to (276.3, 79.3), turned to 90 degrees
- moved R28 20.8 mm to (297.5, 60.3), turned to 0 degrees
- moved J63 19.8 mm to (297.0, 71.3), turned to 270 degrees
- moved C13 19.8 mm to (289.4, 103.9), turned to 180 degrees
- moved C15 19.8 mm to (289.2, 124.1), turned to 180 degrees
- moved R10 19.4 mm to (283.6, 100.8), turned to 270 degrees
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Routing:
- net +48V: vias 0 -> 1
